File: hardware/6502-retro/6502-retro.kicad_sch (KiCad schematic)
At the start: 35 parts, among them J1 SLOT 1, J2 SLOT 2, J3 SLOT 3, J4 0548190519, J5 Conn_01x03_Male, SW1 RESET, U1 62256 SRAM, U2 28C256 ROM, U3 6551 ACIA, U4 W65C02SxP, U5 AT22V10Q, U6 SN74HC08N, U7 DS1813, X1 2MHz, X2 1.8432MHz

Commit message: updated hardware
Parts:
- R10: value 3.9K -> 4.7
Changed lines of the file:
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@@
   (title_block
     (title "6502-Retro!")
-    (date "2023-07-11")
+    (date "2023-07-18")
     (rev "2.0")
     (company "David Latham")
@@
     (in_bom yes) (on_board yes)
     (property "Reference" "R10" (id 0) (at 247.3295 54.7607 90))
-    (property "Value" "3.9K" (id 1) (at 248.92 52.832 90))
+    (property "Value" "4.7" (id 1) (at 248.92 52.832 90))
     (property "Footprint" "Resistor_THT:R_Axial_DIN0207_L6.3mm_D2.5mm_P7.62mm_Horizontal" (id 2) (at 248.92 51.054 90)
       (effects (font (size 1.27 1.27)) hide)
@@
     )
     (path "/333a7369-36f7-4d4f-9da3-e58a824b2297"
-      (reference "R10") (unit 1) (value "3.9K") (footprint "Resistor_THT:R_Axial_DIN0207_L6.3mm_D2.5mm_P7.62mm_Horizontal")
+      (reference "R10") (unit 1) (value "4.7") (footprint "Resistor_THT:R_Axial_DIN0207_L6.3mm_D2.5mm_P7.62mm_Horizontal")
     )
     (path "/0fd938dd-c70d-40ff-8424-76ff1baf22b5"
