File: hardware/6502-retro-io/6502-retro-io.kicad_pcb (KiCad board)
At the start: 4 copper layers, 100 x 47.4 mm, 24 parts, among them J1 SLOT, J2 Mini-DIN-6, J4 Conn_01x08, J5 Conn_01x03, Q1 2N4401, U1 W65C22SxP, U2 PIC16F628A-IP, Y1 20MHz

Commit message: updated hardware
Parts:
- removed D9: YELLOW, LED_THT:LED_D3.0mm
- removed Q1: 2N4401, Package_TO_SOT_THT:TO-92L_Inline
- removed R1: 1K, Resistor_THT:R_Axial_DIN0207_L6.3mm_D2.5mm_P7.62mm_Horizontal
- removed R2: 10K, Resistor_THT:R_Axial_DIN0207_L6.3mm_D2.5mm_P7.62mm_Horizontal
- moved U2 0.21 mm to (159.8, 100.8)
Connections:
- J2 pad 3: Net-(J2-Pad3) -> GND
- U2 pad 4: /~{RST} -> +5V
Routing:
- net /~{RST}: track 108.9 -> 29.9 mm, vias 4 -> 2
- net /CA1: track 115.5 -> 73.0 mm, vias 5 -> 3
- net Net-(J2-Pad3): track 12.1 -> 0.00 mm
- net Net-(Q1-Pad2): track 7.58 -> 0.00 mm
Other:
- board text added: "6502-Retro-IO (c) David Latham Rev 2.0 - 2023"
- board text removed: "6502-Retro-IO (c) David Latham Rev 1.0 - 2023"
