File: hardware/6502-retro-io/6502-retro-io.kicad_sch (KiCad schematic)
At the start: 24 parts, among them J1 SLOT, J2 Mini-DIN-6, J4 Conn_01x08, J5 Conn_01x03, Q1 2N4401BU, U1 W65C22SxP, U2 PIC16F628A-IP, Y1 20MHz

Commit message: updated hardware
Parts:
- removed D9: YELLOW, LED_THT:LED_D3.0mm, symbol Device:LED_Small
- removed Q1: 2N4401BU, Package_TO_SOT_THT:TO-92L_Inline, symbol dk_Transistors-Bipolar-BJT-Single:2N4401BU
- removed R1: 1K, Resistor_THT:R_Axial_DIN0207_L6.3mm_D2.5mm_P7.62mm_Horizontal, symbol Device:R
- removed R2: 10K, Resistor_THT:R_Axial_DIN0207_L6.3mm_D2.5mm_P7.62mm_Horizontal, symbol Device:R
Connections:
- net +5V: now also U2.4 (~{MCLR}/Vpp/RA5)
- net GND: now also J2.3
- net ~{RST}: no longer U2.4 (~{MCLR}/Vpp/RA5)
Other:
- note added: "LED has current limiting resistors built in"
- note removed: "LEDs have current limiting resistors built in"
